File: hardware/RFPowerMeter.sch (KiCad schematic (older format))
At the start: 36 parts, among them IC1 ATMEGA328-P, P1 SMA, P2 SMA, P3 CONN_01X01, P4 CONN_01X01, SW1 SELECT, U1 7805, U2 AD8307, U3 4056, U4 4056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

Commit message: Improved noise immunity
Parts:
- removed P2: SMA, Pin_Headers:Pin_Header_Straight_1x02, symbol BNC
- added C14: 100µF, Capacitors_ThroughHole:C_Radial_D6.3_L11.2_P2.5, symbol CP
- P1: footprint Pin_Headers:Pin_Header_Straight_1x02 -> (none)
- R3: footprint Resistors_ThroughHole:Resistor_Horizontal_RM15mm -> Wire_Pads:SolderWirePad_single_1-2mmDrill
Connections:
- net 7-13.8V: now also C14.1
- net Earth: now also C14.2
Other:
- moved on the sheet: C2, C9, P1, U1
Changed lines of the file:
@@
 Sheet 1 1
 Title "RF Power Meter 1kW"
-Date "2019-06-07"
-Rev "1"
+Date "2019-06-14"
+Rev "2"
 Comp "juvar.fi"
 Comment1 "Juha-Pekka Varjonen"
@@
 L BNC P1
 U 1 1 5CF92CCE
-P 1000 1650
-F 0 "P1" H 1010 1770 50  0000 C CNN
-F 1 "SMA" V 1110 1590 50  0000 C CNN
-F 2 "Pin_Headers:Pin_Header_Straight_1x02" H 1000 1650 50  0001 C CNN
-F 3 "" H 1000 1650 50  0000 C CNN
-	1    1000 1650
-	-1   0    0    -1
-$EndComp
-$Comp
-L BNC P2
-U 1 1 5CF92D6D
-P 1000 2250
-F 0 "P2" H 1010 2370 50  0000 C CNN
-F 1 "SMA" V 1110 2190 50  0000 C CNN
-F 2 "Pin_Headers:Pin_Header_Straight_1x02" H 1000 2250 50  0001 C CNN
-F 3 "" H 1000 2250 50  0000 C CNN
-	1    1000 2250
+P 1000 1950
+F 0 "P1" H 1010 2070 50  0000 C CNN
+F 1 "SMA" V 1110 1890 50  0000 C CNN
+F 2 "" H 1000 1950 50  0001 C CNN
+F 3 "" H 1000 1950 50  0000 C CNN
+	1    1000 1950
 	-1   0    0    -1
 $EndComp
@@
 F 0 "R3" V 1530 1950 50  0000 C CNN
 F 1 "100k" V 1450 1950 50  0000 C CNN
-F 2 "Resistors_ThroughHole:Resistor_Horizontal_RM15mm" V 1380 1950 50  0001 C CNN
+F 2 "Wire_Pads:SolderWirePad_single_1-2mmDrill" V 1380 1950 50  0001 C CNN
 F 3 "" H 1450 1950 50  0000 C CNN
 	1    1450 1950
@@
 L C C9
 U 1 1 5CF9350F
-P 2500 5350
-F 0 "C9" H 2525 5450 50  0000 L CNN
-F 1 "100nF" H 2525 5250 50  0000 L CNN
-F 2 "Capacitors_ThroughHole:C_Disc_D3_P2.5" H 2538 5200 50  0001 C CNN
-F 3 "" H 2500 5350 50  0000 C CNN
-	1    2500 5350
+P 2550 5350
+F 0 "C9" H 2575 5450 50  0000 L CNN
+F 1 "100nF" H 2575 5250 50  0000 L CNN
+F 2 "Capacitors_ThroughHole:C_Disc_D3_P2.5" H 2588 5200 50  0001 C CNN
+F 3 "" H 2550 5350 50  0000 C CNN
+	1    2550 5350
 	1    0    0    -1
 $EndComp
@@
 L C C2
 U 1 1 5CF9357B
-P 1400 5350
-F 0 "C2" H 1425 5450 50  0000 L CNN
-F 1 "330nF" H 1425 5250 50  0000 L CNN
-F 2 "Capacitors_ThroughHole:C_Disc_D3_P2.5" H 1438 5200 50  0001 C CNN
-F 3 "" H 1400 5350 50  0000 C CNN
-	1    1400 5350
+P 1650 5350
+F 0 "C2" H 1675 5450 50  0000 L CNN
+F 1 "330nF" H 1675 5250 50  0000 L CNN
+F 2 "Capacitors_ThroughHole:C_Disc_D3_P2.5" H 1688 5200 50  0001 C CNN
+F 3 "" H 1650 5350 50  0000 C CNN
+	1    1650 5350
 	1    0    0    -1
 $EndComp
@@
 L GND #PWR04
 U 1 1 5CF9361F
-P 2500 6050
-F 0 "#PWR04" H 2500 5800 50  0001 C CNN
-F 1 "GND" H 2500 5900 50  0000 C CNN
-F 2 "" H 2500 6050 50  0000 C CNN
-F 3 "" H 2500 6050 50  0000 C CNN
-	1    2500 6050
+P 2550 6050
+F 0 "#PWR04" H 2550 5800 50  0001 C CNN
+F 1 "GND" H 2550 5900 50  0000 C CNN
+F 2 "" H 2550 6050 50  0000 C CNN
+F 3 "" H 2550 6050 50  0000 C CNN
+	1    2550 6050
 	1    0    0    -1
 $EndComp
@@
 L GND #PWR05
 U 1 1 5CF9364B
-P 1400 6050
-F 0 "#PWR05" H 1400 5800 50  0001 C CNN
-F 1 "GND" H 1400 5900 50  0000 C CNN
-F 2 "" H 1400 6050 50  0000 C CNN
-F 3 "" H 1400 6050 50  0000 C CNN
-	1    1400 6050
+P 1650 6050
+F 0 "#PWR05" H 1650 5800 50  0001 C CNN
+F 1 "GND" H 1650 5900 50  0000 C CNN
+F 2 "" H 1650 6050 50  0000 C CNN
+F 3 "" H 1650 6050 50  0000 C CNN
+	1    1650 6050
 	1    0    0    -1
 $EndComp
@@
 L GND #PWR06
 U 1 1 5CF936F8
-P 1950 6050
-F 0 "#PWR06" H 1950 5800 50  0001 C CNN
-F 1 "GND" H 1950 5900 50  0000 C CNN
-F 2 "" H 1950 6050 50  0000 C CNN
-F 3 "" H 1950 6050 50  0000 C CNN
-	1    1950 6050
+P 2100 6050
+F 0 "#PWR06" H 2100 5800 50  0001 C CNN
+F 1 "GND" H 2100 5900 50  0000 C CNN
+F 2 "" H 2100 6050 50  0000 C CNN
+F 3 "" H 2100 6050 50  0000 C CNN
+	1    2100 6050
 	1    0    0    -1
 $EndComp
@@
 L +5V #PWR07
 U 1 1 5CF93DF5
-P 2500 4900
-F 0 "#PWR07" H 2500 4750 50  0001 C CNN
-F 1 "+5V" H 2500 5040 50  0000 C CNN
-F 2 "" H 2500 4900 50  0000 C CNN
-F 3 "" H 2500 4900 50  0000 C CNN
-	1    2500 4900
+P 2550 4900
+F 0 "#PWR07" H 2550 4750 50  0001 C CNN
+F 1 "+5V" H 2550 5040 50  0000 C CNN
+F 2 "" H 2550 4900 50  0000 C CNN
+F 3 "" H 2550 4900 50  0000 C CNN
+	1    2550 4900
 	1    0    0    -1
 $EndComp
@@
 L VSS #PWR013
 U 1 1 5CFA097F
-P 1650 5950
-F 0 "#PWR013" H 1650 5800 50  0001 C CNN
-F 1 "VSS" H 1650 6100 50  0000 C CNN
-F 2 "" H 1650 5950 50  0000 C CNN
-F 3 "" H 1650 5950 50  0000 C CNN
-	1    1650 5950
+P 2300 5950
+F 0 "#PWR013" H 2300 5800 50  0001 C CNN
+F 1 "VSS" H 2300 6100 50  0000 C CNN
+F 2 "" H 2300 5950 50  0000 C CNN
+F 3 "" H 2300 5950 50  0000 C CNN
+	1    2300 5950
 	1    0    0    -1
 $EndComp
@@
 L Earth #PWR014
 U 1 1 5CFA09D3
-P 1800 5950
-F 0 "#PWR014" H 1800 5700 50  0001 C CNN
-F 1 "Earth" H 1800 5800 50  0001 C CNN
-F 2 "" H 1800 5950 50  0000 C CNN
-F 3 "" H 1800 5950 50  0000 C CNN
-	1    1800 5950
+P 2450 5950
+F 0 "#PWR014" H 2450 5700 50  0001 C CNN
+F 1 "Earth" H 2450 5800 50  0001 C CNN
+F 2 "" H 2450 5950 50  0000 C CNN
+F 3 "" H 2450 5950 50  0000 C CNN
+	1    2450 5950
 	-1   0    0    1
 $EndComp
@@
 L GND #PWR015
 U 1 1 5CFA0A20
-P 1650 6050
-F 0 "#PWR015" H 1650 5800 50  0001 C CNN
-F 1 "GND" H 1650 5900 50  0000 C CNN
-F 2 "" H 1650 6050 50  0000 C CNN
-F 3 "" H 1650 6050 50  0000 C CNN
-	1    1650 6050
+P 2300 6050
+F 0 "#PWR015" H 2300 5800 50  0001 C CNN
+F 1 "GND" H 2300 5900 50  0000 C CNN
+F 2 "" H 2300 6050 50  0000 C CNN
+F 3 "" H 2300 6050 50  0000 C CNN
+	1    2300 6050
 	1    0    0    -1
 $EndComp
@@
 	2900 6050 2900 5500
 Wire Wire Line
-	1000 1850 1000 1900
-Wire Wire Line
 	1300 1950 1150 1950
-Connection ~ 1150 1950
-Wire Wire Line
-	1400 6050 1400 5500
-Wire Wire Line
-	950  5000 1550 5000
-Wire Wire Line
-	1400 5000 1400 5200
-Wire Wire Line
-	2700 5000 2350 5000
-Wire Wire Line
-	2500 4900 2500 5200
-Wire Wire Line
-	2500 5500 2500 6050
-Wire Wire Line
-	1950 6050 1950 5300
-Connection ~ 2500 5000
-Connection ~ 1400 5000
+Wire Wire Line
+	1650 6050 1650 5500
+Wire Wire Line
+	1650 5000 1650 5200
+Wire Wire Line
+	2550 4900 2550 5200
+Wire Wire Line
+	2550 5500 2550 6050
+Wire Wire Line
+	2100 6050 2100 5300
+Connection ~ 2550 5000
+Connection ~ 1650 5000
 Wire Wire Line
 	2250 2250 2300 2250
@@
 Wire Wire Line
 	700  3300 700  1000
-Wire Wire Line
-	1000 1900 700  1900
-Connection ~ 700  1900
 Connection ~ 2100 3300
 Connection ~ 2100 2900
@@
 Connection ~ 6150 2400
 Wire Wire Line
-	1800 5950 1800 6000
-Wire Wire Line
-	1800 6000 1650 6000
-Wire Wire Line
-	1650 5950 1650 6050
-Connection ~ 1650 6000
+	2450 5950 2450 6000
+Wire Wire Line
+	2450 6000 2300 6000
+Wire Wire Line
+	2300 5950 2300 6050
+Connection ~ 2300 6000
 $Comp
 L VDD #PWR016
 U 1 1 5CFA0BFD
-P 2700 4900
-F 0 "#PWR016" H 2700 4750 50  0001 C CNN
-F 1 "VDD" H 2700 5050 50  0000 C CNN
-F 2 "" H 2700 4900 50  0000 C CNN
-F 3 "" H 2700 4900 50  0000 C CNN
-	1    2700 4900
-	1    0    0    -1
-$EndComp
-Wire Wire Line
-	2700 4900 2700 5000
+P 2750 4900
+F 0 "#PWR016" H 2750 4750 50  0001 C CNN
+F 1 "VDD" H 2750 5050 50  0000 C CNN
+F 2 "" H 2750 4900 50  0000 C CNN
+F 3 "" H 2750 4900 50  0000 C CNN
+	1    2750 4900
+	1    0    0    -1
+$EndComp
+Wire Wire Line
+	2750 5000 2750 4900
 Text Notes 2200 3400 0    60   ~ 0
 SHIELDED
@@
 Text Notes 3900 4500 0    118  ~ 0
 AVR Microcontroller
-Text Notes 1300 4500 0    118  ~ 0
+Text Notes 1150 4500 0    118  ~ 0
 Power Supply
 $Comp
@@
 Text Notes 2400 2350 0    60   ~ 0
 +/-3dB
-Wire Wire Line
-	1000 2450 1000 2500
-Wire Wire Line
-	1000 2500 700  2500
-Connection ~ 700  2500
-Wire Wire Line
-	1150 1650 1150 2250
 $Comp
 L 7805 U1
 U 1 1 5CFAA838
-P 1950 5050
-F 0 "U1" H 2100 4854 50  0000 C CNN
-F 1 "7805" H 1950 5250 50  0000 C CNN
-F 2 "TO_SOT_Packages_THT:TO-220_Neutral123_Horizontal" H 1950 5050 50  0001 C CNN
-F 3 "" H 1950 5050 50  0000 C CNN
-	1    1950 5050
+P 2100 5050
+F 0 "U1" H 2250 4854 50  0000 C CNN
+F 1 "7805" H 2100 5250 50  0000 C CNN
+F 2 "TO_SOT_Packages_THT:TO-220_Neutral123_Horizontal" H 2100 5050 50  0001 C CNN
+F 3 "" H 2100 5050 50  0000 C CNN
+	1    2100 5050
 	1    0    0    -1
 $EndComp
@@
 Wire Wire Line
 	5650 5100 5600 5100
+Wire Wire Line
+	1000 2150 1000 2200
+Wire Wire Line
+	1000 2200 700  2200
+Connection ~ 700  2200
+Wire Wire Line
+	2500 5000 2750 5000
+Wire Wire Line
+	950  5000 1700 5000
+$Comp
+L CP C14
+U 1 1 5D030CB0
+P 1350 5350
+F 0 "C14" H 1375 5450 50  0000 L CNN
+F 1 "100µF" H 1375 5250 50  0000 L CNN
+F 2 "Capacitors_ThroughHole:C_Radial_D6.3_L11.2_P2.5" H 1388 5200 50  0001 C CNN
+F 3 "" H 1350 5350 50  0000 C CNN
+	1    1350 5350
+	1    0    0    -1
+$EndComp
+$Comp
+L GND #PWR027
+U 1 1 5D030E3B
+P 1350 6050
+F 0 "#PWR027" H 1350 5800 50  0001 C CNN
+F 1 "GND" H 1350 5900 50  0000 C CNN
+F 2 "" H 1350 6050 50  0000 C CNN
+F 3 "" H 1350 6050 50  0000 C CNN
+	1    1350 6050
+	1    0    0    -1
+$EndComp
+Wire Wire Line
+	1350 6050 1350 5500
+Wire Wire Line
+	1350 5200 1350 5000
+Connection ~ 1350 5000
 $EndSCHEMATC

Commit message: Improved noice immunity, fixed hole sizes
Parts:
- added C15: 100nF, Capacitors_ThroughHole:C_Disc_D3_P2.5, symbol C
Connections:
- net Earth: now also C15.2
- net at IC1.19 ((PCINT5/SCK)PB5), SW1.1: now also C15.1
Other:
- note added: "Internal pull-up loads capacitor"
Changed lines of the file:
@@
 $EndComp
 Wire Wire Line
-	7400 5600 7400 5500
+	7400 5150 7400 5600
 Wire Wire Line
 	7400 5500 7350 5500
@@
 	1350 5200 1350 5000
 Connection ~ 1350 5000
+$Comp
+L C C15
+U 1 1 5D04A764
+P 7050 5150
+F 0 "C15" H 7075 5250 50  0000 L CNN
+F 1 "100nF" H 7075 5050 50  0000 L CNN
+F 2 "Capacitors_ThroughHole:C_Disc_D3_P2.5" H 7088 5000 50  0001 C CNN
+F 3 "" H 7050 5150 50  0000 C CNN
+	1    7050 5150
+	0    -1   -1   0
+$EndComp
+Wire Wire Line
+	6900 5150 6700 5150
+Wire Wire Line
+	6700 5150 6700 5500
+Connection ~ 6700 5500
+Wire Wire Line
+	7200 5150 7400 5150
+Connection ~ 7400 5500
+Text Notes 6200 4800 0    60   ~ 0
+Internal pull-up loads capacitor
 $EndSCHEMATC
